Commit message: Update front_boundary_lu.urdf

File: assets/up/front_boundary_lu.urdf (robot description, URDF)
Before this commit: robot back_boundary, 1 links, 0 joints
Links:
- link back_wall: geometry collision box size=3 0.1 0.5; visual box size=3 0.1 0.5

Commit message: Update front_boundary_lu.urdf

File: assets/up/front_boundary_lu.urdf (robot description, URDF)
Before this commit: robot back_boundary, 1 links, 0 joints
Links:
- link back_wall: geometry collision box size=3.3 0.1 0.5; visual box size=3.3 0.1 0.5
