Commit message: Update side_boundary_rd.urdf

File: assets/down/side_boundary_rd.urdf (robot description, URDF)
Before this commit: robot side_boundaries, 1 links, 0 joints
Links:
- link side_wall: geometry collision box size=0.1 1.6 0.5; visual box size=0.1 1.6 0.5

Commit message: Update side_boundary_rd.urdf

File: assets/down/side_boundary_rd.urdf (robot description, URDF)
Before this commit: robot side_boundaries, 1 links, 0 joints
Links:
- link side_wall: geometry collision box size=0.1 1.253 0.5; visual box size=0.1 1.253 0.5
