Commit message: Update front_boundary_ld.urdf

File: assets/down/front_boundary_ld.urdf (robot description, URDF)
Before this commit: robot back_boundary, 1 links, 0 joints
Links:
- link back_wall: geometry collision box size=2.1 0.1 0.5; visual box size=2.1 0.1 0.5

Commit message: Update front_boundary_ld.urdf

File: assets/down/front_boundary_ld.urdf (robot description, URDF)
Before this commit: robot back_boundary, 1 links, 0 joints
Links:
- link back_wall: geometry collision box size=2.3 0.1 0.5; visual box size=2.3 0.1 0.5
